Commit message: (fix)删去了一些不必要的文件

File: src/ur_driver/src/ur5_description/urdf/ur.ros2_control.xacro (robot description, xacro)
@@ -1,10 +1,8 @@
 <?xml version="1.0"?>
 <robot xmlns:xacro="http://www.ros.org/wiki/xacro">
-  <xacro:include filename="$(find ur5_description)/urdf/robotiq_arg2f_transmission.xacro" />
-  <xacro:robotiq_arg2f_transmission prefix="${tf_prefix}"/>
   <xacro:macro name="ur_ros2_control" params="
     name
-    use_fake_hardware:=true fake_sensor_commands:=false
-    sim_gazebo:=true
+    use_fake_hardware:=false fake_sensor_commands:=false
+    sim_gazebo:=false
     sim_ignition:=false
     headless_mode:=false

File: src/ur_driver/src/ur5_description/urdf/ur.urdf.xacro (robot description, xacro)
@@ -4,14 +4,14 @@
    <xacro:arg name="name" default="ur"/>
    <!-- import main macro -->
-   <xacro:include filename="$(find ur5_description)/urdf/ur_macro.xacro"/>
+   <xacro:include filename="$(find ur_description)/urdf/ur_macro.xacro"/>
    <!-- possible 'ur_type' values: ur3, ur3e, ur5, ur5e, ur7e, ur10, ur10e, ur12e, ur16e, ur15, ur20, ur30 -->
    <!-- the default value should raise an error in case this was called without defining the type -->
-   <xacro:arg name="ur_type" default="ur5"/>
+   <xacro:arg name="ur_type" default="ur5x"/>
    <!-- parameters -->
    <xacro:arg name="tf_prefix" default="" />
-   <xacro:arg name="joint_limit_params" default="$(find ur5_description)/config/$(arg ur_type)/joint_limits.yaml"/>
-   <xacro:arg name="kinematics_params" default="$(find ur5_description)/config/$(arg ur_type)/default_kinematics.yaml"/>
-   <xacro:arg name="physical_params" default="$(find ur5_description)/config/$(arg ur_type)/physical_parameters.yaml"/>
-   <xacro:arg name="visual_params" default="$(find ur5_description)/config/$(arg ur_type)/visual_parameters.yaml"/>
+   <xacro:arg name="joint_limit_params" default="$(find ur_description)/config/$(arg ur_type)/joint_limits.yaml"/>
+   <xacro:arg name="kinematics_params" default="$(find ur_description)/config/$(arg ur_type)/default_kinematics.yaml"/>
+   <xacro:arg name="physical_params" default="$(find ur_description)/config/$(arg ur_type)/physical_parameters.yaml"/>
+   <xacro:arg name="visual_params" default="$(find ur_description)/config/$(arg ur_type)/visual_parameters.yaml"/>
    <xacro:arg name="transmission_hw_interface" default=""/>
    <xacro:arg name="safety_limits" default="false"/>
@@ -40,11 +40,11 @@
    <xacro:arg name="tool_tcp_port" default="54321" />
      <!-- Simulation parameters -->
-   <xacro:arg name="use_fake_hardware" default="true" />
+   <xacro:arg name="use_fake_hardware" default="false" />
    <xacro:arg name="fake_sensor_commands" default="false" />
-   <xacro:arg name="sim_gazebo" default="true" />
+   <xacro:arg name="sim_gazebo" default="false" />
    <xacro:arg name="sim_ignition" default="false" />
-   <xacro:arg name="simulation_controllers" default="$(find gazebo_driver)/config/ur_controllers.yaml" />
+   <xacro:arg name="simulation_controllers" default="" />
    <!-- initial position for simulations (Fake Hardware, Gazebo, Ignition) -->
-   <xacro:arg name="initial_positions_file" default="$(find ur5_description)/config/initial_positions.yaml"/>
+   <xacro:arg name="initial_positions_file" default="$(find ur_description)/config/initial_positions.yaml"/>
    <!-- convert to property to use substitution in function -->
    <xacro:property name="initial_positions_file" default="$(arg initial_positions_file)"/>

File: src/ur_driver/src/ur5_description/urdf/ur_macro.xacro (robot description, xacro)
@@ -42,7 +42,6 @@
      - Muhammad Asif Rana
   -->
-  <xacro:include filename="$(find ur5_description)/urdf/inc/ur_transmissions.xacro" />
-  <xacro:include filename="$(find ur5_description)/urdf/inc/ur_common.xacro" />
-  <xacro:include filename="$(find ur5_description)/urdf/robotiq_arg2f_85_model_macro.xacro" />
+  <xacro:include filename="$(find ur_description)/urdf/inc/ur_transmissions.xacro" />
+  <xacro:include filename="$(find ur_description)/urdf/inc/ur_common.xacro" />
   <xacro:macro name="ur_robot" params="
     name
@@ -95,5 +94,5 @@
     <xacro:if value="${generate_ros2_control_tag}">
       <!-- ros2 control include -->
-      <xacro:include filename="$(find ur5_description)/urdf/ur.ros2_control.xacro" />
+      <xacro:include filename="$(find ur_description)/urdf/ur.ros2_control.xacro" />
       <!-- ros2 control instance -->
       <xacro:ur_ros2_control
@@ -437,18 +436,10 @@
       <origin xyz="0 0 0" rpy="0 ${-pi/2.0} ${-pi/2.0}" />
     </joint>
-    <xacro:include filename="$(find ur5_description)/urdf/robotiq_arg2f_85_model_macro.xacro"/>
-    <xacro:robotiq_arg2f_85 prefix="${tf_prefix}"/>
-    <!-- 连接夹爪到 flange -->
-    <joint name="${tf_prefix}flange_to_gripper" type="fixed">
-      <parent link="${tf_prefix}flange"/>
-      <child link="${tf_prefix}robotiq_arg2f_base_link"/>
-      <origin xyz="0 0 0" rpy="${pi/2.0} 0 ${pi/2.0}"/>
-    </joint>
     <!-- ROS-Industrial 'tool0' frame - all-zeros tool frame -->
     <link name="${tf_prefix}tool0"/>
-    <joint name="${tf_prefix}gripper-to-tool0" type="fixed">
+    <joint name="${tf_prefix}flange-tool0" type="fixed">
       <!-- default toolframe - X+ left, Y+ up, Z+ front -->
       <origin xyz="0 0 0" rpy="${pi/2.0} 0 ${pi/2.0}"/>
-      <parent link="${tf_prefix}left_inner_finger_pad"/>
+      <parent link="${tf_prefix}flange"/>
       <child link="${tf_prefix}tool0"/>
     </joint>
