Commit message: (feat)修改参数文件，解决碰撞问题，能够正常进行路径规划

File: src/ur_driver/src/moveit_driver/srdf/ur.srdf.xacro (robot description, xacro)
@@ -5,5 +5,5 @@
   <!-- parameters -->
   <xacro:arg name="prefix" default="" />
-  <xacro:include filename="$(find ur_moveit_config)/srdf/ur_macro.srdf.xacro"/>
+  <xacro:include filename="$(find moveit_driver)/srdf/ur_macro.srdf.xacro"/>
   <xacro:ur_srdf name="$(arg name)" prefix="$(arg prefix)"/>
 </robot>

File: src/ur_driver/src/moveit_driver/srdf/ur_macro.srdf.xacro (robot description, xacro)
@@ -13,4 +13,17 @@
     <group name="${prefix}${name}_manipulator">
       <chain base_link="${prefix}base_link" tip_link="${prefix}tool0" />
+    </group>
+    <!-- ============= 添加夹爪规划组 ============= -->
+    <group name="${prefix}gripper">
+      <joint name="${prefix}finger_joint" />
+      <!-- joint name="${prefix}left_inner_knuckle_joint" />
+      <joint name="${prefix}left_inner_finger_joint" />
+      <joint name="${prefix}right_inner_knuckle_joint" />
+      <joint name="${prefix}right_inner_finger_joint" /-->
+    </group>
+    <!-- arm & gripper -->
+    <group name="${prefix}arm_with_gripper">
+      <group name="${prefix}${name}_manipulator" />
+      <group name="${prefix}gripper" />
     </group>
     <!--GROUP STATES - Purpose - Define a named state for a particular group, in terms of joint values. This is useful to define states like 'folded arms'-->
@@ -39,4 +52,21 @@
       <joint name="${prefix}wrist_3_joint" value="-0.11" />
     </group_state>
+    <!-- ============= 添加夹爪状态 ============= -->
+    <group_state name="${prefix}gripper_open" group="${prefix}gripper">
+      <joint name="${prefix}finger_joint" value="0.04" />
+    </group_state>
+    <group_state name="${prefix}gripper_closed" group="${prefix}gripper">
+      <joint name="${prefix}finger_joint" value="0.0" />
+    </group_state>
+    <!-- arm & gripper -->
+    <group_state name="${prefix}home_with_gripper_open" group="${prefix}arm_with_gripper">
+      <joint name="${prefix}elbow_joint" value="0" />
+      <joint name="${prefix}shoulder_lift_joint" value="-1.5707" />
+      <joint name="${prefix}shoulder_pan_joint" value="0" />
+      <joint name="${prefix}wrist_1_joint" value="0" />
+      <joint name="${prefix}wrist_2_joint" value="0" />
+      <joint name="${prefix}wrist_3_joint" value="0" />
+      <joint name="${prefix}finger_joint" value="0.04" />
+    </group_state>
     <!--END EFFECTOR - Purpose - Represent information about an end effector.-->
     <!--VIRTUAL JOINT - Purpose - this element defines a virtual joint between a robot link and an external frame of reference (considered fixed with respect to the robot)-->
@@ -53,4 +83,62 @@
     <disable_collisions link1="${prefix}wrist_1_link" link2="${prefix}wrist_3_link" reason="Never" />
     <disable_collisions link1="${prefix}wrist_2_link" link2="${prefix}wrist_3_link" reason="Adjacent" />
+    <disable_collisions link1="${prefix}wrist_3_link" link2="${prefix}robotiq_arg2f_base_link" reason="Adjacent"/>
+    <!-- ============= 添加夹爪碰撞忽略 ============= -->
+    <!-- 夹爪枚举，没招了。。。 -->
+    <disable_collisions link1="${prefix}robotiq_arg2f_base_link" link2="${prefix}left_outer_knuckle" reason="Never"/>
+    <disable_collisions link1="${prefix}robotiq_arg2f_base_link" link2="${prefix}left_inner_knuckle" reason="Never"/>
+    <disable_collisions link1="${prefix}robotiq_arg2f_base_link" link2="${prefix}right_outer_knuckle" reason="Never"/>
+    <disable_collisions link1="${prefix}robotiq_arg2f_base_link" link2="${prefix}right_inner_knuckle" reason="Never"/>
+    <disable_collisions link1="${prefix}robotiq_arg2f_base_link" link2="${prefix}left_outer_finger" reason="Never"/>
+    <disable_collisions link1="${prefix}robotiq_arg2f_base_link" link2="${prefix}right_outer_finger" reason="Never"/>
+    <disable_collisions link1="${prefix}robotiq_arg2f_base_link" link2="${prefix}left_inner_finger" reason="Never"/>
+    <disable_collisions link1="${prefix}robotiq_arg2f_base_link" link2="${prefix}right_inner_finger" reason="Never"/>
+    <disable_collisions link1="${prefix}robotiq_arg2f_base_link" link2="${prefix}left_inner_finger_pad" reason="Never"/>
+    <disable_collisions link1="${prefix}robotiq_arg2f_base_link" link2="${prefix}right_inner_finger_pad" reason="Never"/>
+    <disable_collisions link1="${prefix}left_outer_knuckle" link2="${prefix}left_inner_knuckle" reason="Never"/>
+    <disable_collisions link1="${prefix}left_outer_knuckle" link2="${prefix}right_outer_knuckle" reason="Never"/>
+    <disable_collisions link1="${prefix}left_outer_knuckle" link2="${prefix}right_inner_knuckle" reason="Never"/>
+    <disable_collisions link1="${prefix}left_outer_knuckle" link2="${prefix}left_outer_finger" reason="Never"/>
+    <disable_collisions link1="${prefix}left_outer_knuckle" link2="${prefix}right_outer_finger" reason="Never"/>
+    <disable_collisions link1="${prefix}left_outer_knuckle" link2="${prefix}left_inner_finger" reason="Never"/>
+    <disable_collisions link1="${prefix}left_outer_knuckle" link2="${prefix}right_inner_finger" reason="Never"/>
+    <disable_collisions link1="${prefix}left_outer_knuckle" link2="${prefix}left_inner_finger_pad" reason="Never"/>
+    <disable_collisions link1="${prefix}left_outer_knuckle" link2="${prefix}right_inner_finger_pad" reason="Never"/>
+    <disable_collisions link1="${prefix}left_inner_knuckle" link2="${prefix}right_outer_knuckle" reason="Never"/>
+    <disable_collisions link1="${prefix}left_inner_knuckle" link2="${prefix}right_inner_knuckle" reason="Never"/>
+    <disable_collisions link1="${prefix}left_inner_knuckle" link2="${prefix}left_outer_finger" reason="Never"/>
+    <disable_collisions link1="${prefix}left_inner_knuckle" link2="${prefix}right_outer_finger" reason="Never"/>
+    <disable_collisions link1="${prefix}left_inner_knuckle" link2="${prefix}left_inner_finger" reason="Never"/>
+    <disable_collisions link1="${prefix}left_inner_knuckle" link2="${prefix}right_inner_finger" reason="Never"/>
+    <disable_collisions link1="${prefix}left_inner_knuckle" link2="${prefix}left_inner_finger_pad" reason="Never"/>
+    <disable_collisions link1="${prefix}left_inner_knuckle" link2="${prefix}right_inner_finger_pad" reason="Never"/>
+    <disable_collisions link1="${prefix}right_outer_knuckle" link2="${prefix}right_inner_knuckle" reason="Never"/>
+    <disable_collisions link1="${prefix}right_outer_knuckle" link2="${prefix}left_outer_finger" reason="Never"/>
+    <disable_collisions link1="${prefix}right_outer_knuckle" link2="${prefix}right_outer_finger" reason="Never"/>
+    <disable_collisions link1="${prefix}right_outer_knuckle" link2="${prefix}left_inner_finger" reason="Never"/>
+    <disable_collisions link1="${prefix}right_outer_knuckle" link2="${prefix}right_inner_finger" reason="Never"/>
+    <disable_collisions link1="${prefix}right_outer_knuckle" link2="${prefix}left_inner_finger_pad" reason="Never"/>
+    <disable_collisions link1="${prefix}right_outer_knuckle" link2="${prefix}right_inner_finger_pad" reason="Never"/>
+    <disable_collisions link1="${prefix}right_inner_knuckle" link2="${prefix}left_outer_finger" reason="Never"/>
+    <disable_collisions link1="${prefix}right_inner_knuckle" link2="${prefix}right_outer_finger" reason="Never"/>
+    <disable_collisions link1="${prefix}right_inner_knuckle" link2="${prefix}left_inner_finger" reason="Never"/>
+    <disable_collisions link1="${prefix}right_inner_knuckle" link2="${prefix}right_inner_finger" reason="Never"/>
+    <disable_collisions link1="${prefix}right_inner_knuckle" link2="${prefix}left_inner_finger_pad" reason="Never"/>
+    <disable_collisions link1="${prefix}right_inner_knuckle" link2="${prefix}right_inner_finger_pad" reason="Never"/>
+    <disable_collisions link1="${prefix}left_outer_finger" link2="${prefix}right_outer_finger" reason="Never"/>
+    <disable_collisions link1="${prefix}left_outer_finger" link2="${prefix}left_inner_finger" reason="Never"/>
+    <disable_collisions link1="${prefix}left_outer_finger" link2="${prefix}right_inner_finger" reason="Never"/>
+    <disable_collisions link1="${prefix}left_outer_finger" link2="${prefix}left_inner_finger_pad" reason="Never"/>
+    <disable_collisions link1="${prefix}left_outer_finger" link2="${prefix}right_inner_finger_pad" reason="Never"/>
+    <disable_collisions link1="${prefix}right_outer_finger" link2="${prefix}left_inner_finger" reason="Never"/>
+    <disable_collisions link1="${prefix}right_outer_finger" link2="${prefix}right_inner_finger" reason="Never"/>
+    <disable_collisions link1="${prefix}right_outer_finger" link2="${prefix}left_inner_finger_pad" reason="Never"/>
+    <disable_collisions link1="${prefix}right_outer_finger" link2="${prefix}right_inner_finger_pad" reason="Never"/>
+    <disable_collisions link1="${prefix}left_inner_finger" link2="${prefix}right_inner_finger" reason="Never"/>
+    <disable_collisions link1="${prefix}left_inner_finger" link2="${prefix}left_inner_finger_pad" reason="Never"/>
+    <disable_collisions link1="${prefix}left_inner_finger" link2="${prefix}right_inner_finger_pad" reason="Never"/>
+    <disable_collisions link1="${prefix}right_inner_finger" link2="${prefix}left_inner_finger_pad" reason="Never"/>
+    <disable_collisions link1="${prefix}right_inner_finger" link2="${prefix}right_inner_finger_pad" reason="Never"/>
+    <disable_collisions link1="${prefix}left_inner_finger_pad" link2="${prefix}right_inner_finger_pad" reason="Never"/>
   </xacro:macro>
 </robot>

File: src/ur_driver/src/ur5_description/urdf/ur.urdf.xacro (robot description, xacro)
@@ -7,5 +7,5 @@
    <!-- possible 'ur_type' values: ur3, ur3e, ur5, ur5e, ur7e, ur10, ur10e, ur12e, ur16e, ur15, ur20, ur30 -->
    <!-- the default value should raise an error in case this was called without defining the type -->
-   <xacro:arg name="ur_type" default="ur5x"/>
+   <xacro:arg name="ur_type" default="ur5"/>
    <!-- parameters -->
    <xacro:arg name="tf_prefix" default="" />

File: src/ur_driver/src/ur5_description/urdf/ur_macro.xacro (robot description, xacro)
@@ -47,8 +47,8 @@
   <xacro:include filename="$(find ur5_description)/urdf/robotiq_arg2f_85_model_macro.xacro" />
     <!-- 添加夹爪参数 -->
-  <xacro:arg name="use_gripper" default="false"/>
+  <xacro:arg name="use_gripper" default="true"/>
   <xacro:arg name="gripper_offset_x" default="0.0"/>
   <xacro:arg name="gripper_offset_y" default="0.0"/>
-  <xacro:arg name="gripper_offset_z" default="0.02"/>
+  <xacro:arg name="gripper_offset_z" default="0.0"/>
   <xacro:arg name="gripper_roll" default="0.0"/>
   <xacro:arg name="gripper_pitch" default="0.0"/>
