Commit message: (feat)修改了urdf文件，按照官方文件集成机械臂

File: src/ur_driver/src/moveit_driver/srdf/ur_macro.srdf.xacro (robot description, xacro)
@@ -14,16 +14,6 @@
       <chain base_link="${prefix}base_link" tip_link="${prefix}tool0" />
     </group>
-    <!-- ============= 添加夹爪规划组 ============= -->
     <group name="${prefix}gripper">
       <joint name="${prefix}finger_joint" />
-      <!-- joint name="${prefix}left_inner_knuckle_joint" />
-      <joint name="${prefix}left_inner_finger_joint" />
-      <joint name="${prefix}right_inner_knuckle_joint" />
-      <joint name="${prefix}right_inner_finger_joint" /-->
-    </group>
-    <!-- arm & gripper -->
-    <group name="${prefix}arm_with_gripper">
-      <group name="${prefix}${name}_manipulator" />
-      <group name="${prefix}gripper" />
     </group>
     <!--GROUP STATES - Purpose - Define a named state for a particular group, in terms of joint values. This is useful to define states like 'folded arms'-->
@@ -35,4 +25,5 @@
       <joint name="${prefix}wrist_2_joint" value="0" />
       <joint name="${prefix}wrist_3_joint" value="0" />
+      <joint name="${prefix}finger_joint" value="0" />
     </group_state>
     <group_state name="${prefix}up" group="${prefix}${name}_manipulator">
@@ -43,4 +34,5 @@
       <joint name="${prefix}wrist_2_joint" value="0" />
       <joint name="${prefix}wrist_3_joint" value="0" />
+      <joint name="${prefix}finger_joint" value="0" />
     </group_state>
     <group_state name="${prefix}test_configuration" group="${prefix}${name}_manipulator">
@@ -51,21 +43,11 @@
       <joint name="${prefix}wrist_2_joint" value="-1.6" />
       <joint name="${prefix}wrist_3_joint" value="-0.11" />
+      <joint name="${prefix}finger_joint" value="0" />
     </group_state>
-    <!-- ============= 添加夹爪状态 ============= -->
     <group_state name="${prefix}gripper_open" group="${prefix}gripper">
-      <joint name="${prefix}finger_joint" value="0.04" />
+      <joint name="${prefix}finger_joint" value="0.0" />
     </group_state>
     <group_state name="${prefix}gripper_closed" group="${prefix}gripper">
-      <joint name="${prefix}finger_joint" value="0.0" />
-    </group_state>
-    <!-- arm & gripper -->
-    <group_state name="${prefix}home_with_gripper_open" group="${prefix}arm_with_gripper">
-      <joint name="${prefix}elbow_joint" value="0" />
-      <joint name="${prefix}shoulder_lift_joint" value="-1.5707" />
-      <joint name="${prefix}shoulder_pan_joint" value="0" />
-      <joint name="${prefix}wrist_1_joint" value="0" />
-      <joint name="${prefix}wrist_2_joint" value="0" />
-      <joint name="${prefix}wrist_3_joint" value="0" />
-      <joint name="${prefix}finger_joint" value="0.04" />
+      <joint name="${prefix}finger_joint" value="0.8" />
     </group_state>
     <!--END EFFECTOR - Purpose - Represent information about an end effector.-->

File: src/ur_driver/src/ur5_description/urdf/ur.ros2_control.xacro (robot description, xacro)
@@ -5,6 +5,6 @@
   <xacro:macro name="ur_ros2_control" params="
     name
-    use_fake_hardware:=false fake_sensor_commands:=false
-    sim_gazebo:=false
+    use_fake_hardware:=true fake_sensor_commands:=false
+    sim_gazebo:=true
     sim_ignition:=false
     headless_mode:=false

File: src/ur_driver/src/ur5_description/urdf/ur.urdf.xacro (robot description, xacro)
@@ -40,9 +40,9 @@
    <xacro:arg name="tool_tcp_port" default="54321" />
      <!-- Simulation parameters -->
-   <xacro:arg name="use_fake_hardware" default="false" />
+   <xacro:arg name="use_fake_hardware" default="true" />
    <xacro:arg name="fake_sensor_commands" default="false" />
-   <xacro:arg name="sim_gazebo" default="false" />
+   <xacro:arg name="sim_gazebo" default="true" />
    <xacro:arg name="sim_ignition" default="false" />
-   <xacro:arg name="simulation_controllers" default="" />
+   <xacro:arg name="simulation_controllers" default="$(find gazebo_driver)/config/ur_controllers.yaml" />
    <!-- initial position for simulations (Fake Hardware, Gazebo, Ignition) -->
    <xacro:arg name="initial_positions_file" default="$(find ur5_description)/config/initial_positions.yaml"/>

File: src/ur_driver/src/ur5_description/urdf/ur_macro.xacro (robot description, xacro)
@@ -44,14 +44,5 @@
   <xacro:include filename="$(find ur5_description)/urdf/inc/ur_transmissions.xacro" />
   <xacro:include filename="$(find ur5_description)/urdf/inc/ur_common.xacro" />
-  <!-- Quoting a new gripper model -->
   <xacro:include filename="$(find ur5_description)/urdf/robotiq_arg2f_85_model_macro.xacro" />
-    <!-- 添加夹爪参数 -->
-  <xacro:arg name="use_gripper" default="true"/>
-  <xacro:arg name="gripper_offset_x" default="0.0"/>
-  <xacro:arg name="gripper_offset_y" default="0.0"/>
-  <xacro:arg name="gripper_offset_z" default="0.0"/>
-  <xacro:arg name="gripper_roll" default="0.0"/>
-  <xacro:arg name="gripper_pitch" default="0.0"/>
-  <xacro:arg name="gripper_yaw" default="0.0"/>
   <xacro:macro name="ur_robot" params="
     name
@@ -446,25 +437,20 @@
       <origin xyz="0 0 0" rpy="0 ${-pi/2.0} ${-pi/2.0}" />
     </joint>
+    <xacro:include filename="$(find ur5_description)/urdf/robotiq_arg2f_85_model_macro.xacro"/>
+    <xacro:robotiq_arg2f_85 prefix="${tf_prefix}"/>
+    <!-- 连接夹爪到 flange -->
+    <joint name="${tf_prefix}flange_to_gripper" type="fixed">
+      <parent link="${tf_prefix}flange"/>
+      <child link="${tf_prefix}robotiq_arg2f_base_link"/>
+      <origin xyz="0 0 0" rpy="${pi/2.0} 0 ${pi/2.0}"/>
+    </joint>
     <!-- ROS-Industrial 'tool0' frame - all-zeros tool frame -->
     <link name="${tf_prefix}tool0"/>
-    <joint name="${tf_prefix}flange-tool0" type="fixed">
+    <joint name="${tf_prefix}gripper-to-tool0" type="fixed">
       <!-- default toolframe - X+ left, Y+ up, Z+ front -->
       <origin xyz="0 0 0" rpy="${pi/2.0} 0 ${pi/2.0}"/>
-      <parent link="${tf_prefix}flange"/>
+      <parent link="${tf_prefix}left_inner_finger_pad"/>
       <child link="${tf_prefix}tool0"/>
     </joint>
-    <!-- ============= 添加夹爪（有条件） ============= -->
-    <xacro:if value="$(arg use_gripper)">
-      <!-- Add Robotiq_85 Claw Model Connection -->
-      <joint name="${tf_prefix}gripper_base_joint" type="fixed">
-        <origin
-          xyz="$(arg gripper_offset_x) $(arg gripper_offset_y) $(arg gripper_offset_z)"
-          rpy="$(arg gripper_roll) $(arg gripper_pitch) $(arg gripper_yaw)"/>
-        <parent link="${tf_prefix}tool0"/>
-        <child link="${tf_prefix}robotiq_arg2f_base_link"/>
-      </joint>
-      <!-- Add Robotiq_85 Claw Body -->
-      <xacro:robotiq_arg2f_85 prefix="${tf_prefix}"/>
-    </xacro:if>
   </xacro:macro>
 </robot>
